File: pcb/main.brd (EAGLE design)
At the start: 160 x 100 mm, 54 parts, among them IC1 NC7SZ14M5X, J3 455-1750-1-ND, J6 M1 connector, J7 M2 connector, Q1 2.5A/30V/105mΩ, U1 LSM303C, U5 ESP-WROOM-32

Commit message: finished schematic (draft1)
Parts:
- removed FB1: (no value), rcl:R0603
- added C21, C22: 10uF, rcl:C0805
- added C23: 0.1uF, electricSheepParty:0603
- added D4: red, electricSheepParty:LED-0603
- added D5: green, electricSheepParty:LED-0603
- added FB2: (no value), rcl:R0603
- added JP1: (no value), pinhead:1X05
- added R11, R12: 330, electricSheepParty:0603
- added TP1, TP10, TP11, TP12, TP13, TP14, TP2, TP3, TP4, TP5, TP6, TP7, TP8, TP9: TPPAD1-17, testpad:P1-17
- added U$5: SC1202-3.3V, carolyn:SOT-223
- moved U5 177.2 mm to (-120.5, -260.8)
- moved C19 167.2 mm to (-40.0, -354.3)
- moved C18 166.8 mm to (-53.1, -355.8)
Connections:
- removed net IO0: U5.25
- new net 3V3M: C10.+, C11.1, C9.+, U$3.4, U$4.P$2
- new net N$20: TP11.TP, U5.17
- new net N$21: TP12.TP, U5.18
- new net N$22: TP13.TP, U5.19
- new net N$25: D4.C, R11.2
- new net N$26: D5.C, R12.2
- new net N$27: TP14.TP, U5.25
- net 3V3: now also C21.1, C23.1, U$5.2, U$5.TAB; no longer C10.+, C11.1, C9.+, U$3.4, U$4.P$2
- net 6V: now also C22.1, U$5.3
- net AGND: now also C22.2, FB2.1, U$5.1; no longer FB1.1
- net GND: now also C21.2, C23.2, FB2.2, JP1.5, R11.1, R12.1; no longer FB1.2
- net N$14: now also TP1.TP
- net N$15: now also TP9.TP
- net N$16: now also D4.A, TP10.TP
- net N$17: now also TP8.TP
- net N$18: now also TP7.TP
- net N$19: now also D5.A, TP6.TP
- net N$23: now also TP5.TP
- net N$24: now also TP4.TP
- net N$4: now also TP2.TP
- net N$5: now also TP3.TP
- net TCK: now also JP1.3
- net TDI: now also JP1.2
- net TDO: now also JP1.4
- net TMS: now also JP1.1

Commit message: layout done! (minus sheep image)
Still need to add sheep and check with tolerances of wherever we fab at,
but otherwise done!!!!
Parts:
- removed C12: 0.1uF, electricSheepParty:0603
- removed R6, R7: 10k, electricSheepParty:0603
- removed U1: LSM303C, SparkFun-Sensors:LGA-12
- added C24: 4.7uF, electricSheepParty:0603
- added IC2: LSM303DLHC, st-microelectronics:LGA-14
- added R13, R14: 10k, electricSheepParty:0603
- added TP15, TP16, TP17, TP20: TPPAD1-13, testpad:P1-13
- C11: value 10uF -> 0.1uF; device rcl:C0805 -> electricSheepParty:0603
- C13: value 0.1uF -> 10uF; device electricSheepParty:0603 -> rcl:C0805
- C14: value 10uF -> 0.22uF; device rcl:C0805 -> electricSheepParty:0603
- R1: value 1M -> 100k
- R8: value 20k -> 2k
- R9: value 10k -> 1k
- TP1, TP10, TP11, TP12, TP13, TP14, TP2, TP3, TP4, TP5, TP6, TP7, TP8, TP9: value TPPAD1-17 -> TPPAD1-13; device testpad:P1-17 -> testpad:P1-13
- moved JP1 445.9 mm to (36.6, 28.5), turned to 180 degrees
- moved R11 428.2 mm to (21.3, 20.8)
- moved R12 423.9 mm to (17.6, 19.6), turned to 270 degrees
- moved TP12 420.6 mm to (38.2, 24.5), turned to 270 degrees
- moved TP13 409.1 mm to (36.8, 22.2), turned to 270 degrees
- moved TP14 406.4 mm to (43.4, 25.3), turned to 90 degrees
- moved TP10 391.4 mm to (7.82, 38.1), turned to 90 degrees
- moved TP9 390.2 mm to (28.5, 21.1), turned to 90 degrees
- moved D4 378.7 mm to (22.1, 17.9), turned to 90 degrees
- moved TP11 377.9 mm to (39.7, 22.3), turned to 270 degrees
- moved D5 377.8 mm to (20.2, 17.9), turned to 90 degrees
- moved C18 372.5 mm to (50.2, 2.08)
- moved C19 370.1 mm to (52.6, 3.96)
- moved TP7 360.0 mm to (33.8, 22.2), turned to 90 degrees
- moved TP6 358.2 mm to (17.6, 16.7), turned to 90 degrees
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Connections:
- removed net INT_MAG: U1.7, U5.29
- removed net INT_XL: U1.12, U5.30
- removed net MAG_RDY: U1.11, U5.28
- removed net N$12: R6.2, R7.1, U1.2, U1.3
- removed net N$6: C12.1, U1.5
- removed net VCC: C18.1, C19.1, IC1.5, U5.2
- new net DAT_RDY: IC2.9, U5.28
- new net INT1: IC2.5, U5.29
- new net INT2: IC2.4, U5.30
- new net N$28: C14.2, IC2.13
- new net N$29: C14.1, IC2.12
- new net N$35: C24.1, IC2.6
- net 3V3: now also C11.1, C18.1, C19.1, IC1.5, IC2.1, IC2.14, R13.1, R14.1, TP16.TP, U5.2; no longer C14.1, C20.1, C3.1, C5.1, R5.2, R7.2, U$2.1, U$2.12, U1.10, U1.9
- net 3V3M: now also C20.1, C3.1, C5.1, R5.2, TP17.TP, U$2.1, U$2.12; no longer C11.1
- net AGND: now also TP10.TP; no longer C11.2
- net GND: now also C11.2, C24.2, IC2.10, IC2.11, IC2.7, TP14.TP; no longer C12.2, C14.2, R6.1, U1.6, U1.8
- net N$14: now also TP3.TP; no longer TP1.TP
- net N$15: now also TP8.TP; no longer TP9.TP
- net N$16: now also TP5.TP; no longer TP10.TP
- net N$17: now also TP7.TP; no longer TP8.TP
- net N$18: now also TP15.TP; no longer TP7.TP
- net N$23: now also TP9.TP; no longer TP5.TP
- net N$27: now also TP20.TP; no longer TP14.TP
- net N$4: now also TP1.TP; no longer TP2.TP
- net N$5: now also TP2.TP; no longer TP3.TP
- net SCL: now also IC2.2, R13.2; no longer U1.1
- net SDA: now also IC2.3, R14.2; no longer U1.4
Routing:
- net 3V3: track 0.00 -> 116.2 mm, vias 0 -> 6
- net AGND: track 0.00 -> 91.7 mm, vias 0 -> 14
- net GND: track 0.00 -> 80.6 mm, vias 0 -> 12
- net PWM_M1A: track 0.00 -> 51.2 mm
- net PWM_SERVO: track 0.00 -> 50.8 mm, vias 0 -> 2
- net PWM_M1B: track 0.00 -> 47.9 mm
- net PWM_M2B: track 0.00 -> 42.5 mm
- net 1/3_BAT: track 0.00 -> 42.0 mm, vias 0 -> 2
- net PWM_M2A: track 0.00 -> 39.6 mm
- net PHOTO: track 0.00 -> 39.1 mm, vias 0 -> 2
- net PWM_LASER: track 0.00 -> 32.9 mm, vias 0 -> 2
- net 3V3M: track 0.00 -> 32.5 mm, vias 0 -> 2
- net SCL: track 0.00 -> 21.0 mm, vias 0 -> 4
- net N$9: track 0.00 -> 16.6 mm, vias 0 -> 2
- net TMS: track 0.00 -> 15.3 mm
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- added copper zone on layer 1, net 3V3
- added copper zone on layer 1, net 3V3M
- added copper zone on layer 1, net 5V
- added copper zone on layer 1, net 6V
- added copper zone on layer 16, net AGND
- added copper zone on layer 16, net GND
- added copper zone on layer 16, net IMU_PROTECT
- added copper zone on layer 1, net N$7
Other:
- board size 160 x 100 mm -> 58 x 52 mm
- board text added: "& Alan Han"
- board text added: "Made by Carolyn Lewelling"
