File: pcb/main.sch (EAGLE design)
At the start: 81 parts, among them IC1 NC7SZ14M5X, IC2 LSM303DLHC, J3 455-1750-1-ND, J6 M1 connector, J7 M2 connector, Q1 2.5A/30V/105mΩ, U5 ESP-WROOM-32

Commit message: editted part layouts. changed pins for uart
Parts:
- removed JP1: (no value), pinhead:PINHD-1X5
- removed TP11, TP2, TP20, TP3, TP4, TP9: TPPAD1-13, testpad:TPPAD1-13
- added C12, C25: 1nF, electricSheepParty:0.1UF-0603-25V-(+80/-20%)
- added J8: (no value), electricSheepParty:CONN_02
- added R6, R7: 470, electricSheepParty:RESISTOR0603
- added RESET2: S2, DiscreteComponents:SWITCH
- added SV1: (no value), con-lsta:FE06-1
- J1: value (none) -> UART header; device electricSheepParty:CONN_02 -> electricSheepParty:CONN_03; COMM Battery Connector -> Servo Connector
- R1: value 100k -> 1M
- R11, R12, R2: value 330 -> 100
Connections:
- removed net N$13: R5.1, U$2.NFAULT
- removed net N$14: TP3.TP, U5.IO35
- removed net N$20: TP11.TP, U5.SD2
- removed net N$23: TP9.TP, U5.IO19
- removed net N$24: TP4.TP, U5.IO23
- removed net N$27: TP20.TP, U5.IO0
- new net BOOT: C25.1, R6.2, R7.2, U5.IO0
- new net NFAULT: R5.1, U$2.NFAULT, U5.SD2
- new net RX: J1.2, U5.RXD0
- new net TX: J1.1, U5.TXD0
- net 3V3: now also R7.1, SV1.1
- net 6V_RAW: now also J8.1; no longer J1.2
- net AGND: now also J8.2; no longer J1.1
- net GND: now also C12.2, C25.2, J1.3, RESET2.P$2, SV1.6, U5.IO12, U5.IO2; no longer JP1.5
- net M1+: now also J6.1; no longer J6.2
- net M1-: now also J6.2; no longer J6.1
- net N$5: now also C12.1, R6.1, RESET2.P$1; no longer TP2.TP, U5.IO34
- net PHOTO: now also U5.IO34; no longer U5.TXD0
- net PWM_LASER: now also U5.IO23; no longer U5.IO2
- net PWM_LED: now also U5.IO27; no longer U5.RXD0
- net PWM_SERVO: now also U5.IO19; no longer U5.IO27
- net TCK: now also SV1.4; no longer JP1.3
- net TDI: now also SV1.3, U5.IO35; no longer JP1.2, U5.IO12
- net TDO: now also SV1.5; no longer JP1.4
- net TMS: now also SV1.2; no longer JP1.1
Other:
- moved on the sheet: R5
